Commit message: format code

File: Raspberry_ros2/description/robot.urdf.xacro (robot description, xacro)
@@ -1,94 +1,94 @@
 <?xml version="1.0"?>
 <robot xmlns:xacro="http://www.ros.org/wiki/xacro" name="test_dd_bot">
-  <xacro:arg name="prefix" default="" />
-  <material name="blue">
-    <color rgba="0.0 0.4 0.8 1"/>
-  </material>
-  <link name="base_link">
-    <visual>
-      <origin xyz="0 0 0.05" rpy="0 0 0"/>
-      <geometry>
-        <box size="0.35 0.22 0.10"/>
-      </geometry>
-      <material name="blue"/>
-    </visual>
-    <collision>
-      <origin xyz="0 0 0.05" rpy="0 0 0"/>
-      <geometry>
-        <box size="0.35 0.22 0.10"/>
-      </geometry>
-    </collision>
-    <inertial>
-      <origin xyz="0 0 0.05" rpy="0 0 0"/>
-      <mass value="2.0"/>
-      <inertia ixx="0.01" ixy="0" ixz="0" iyy="0.02" iyz="0" izz="0.03"/>
-    </inertial>
-  </link>
-  <link name="left_wheel_link">
-    <visual>
-      <origin xyz="0 0 0" rpy="1.5708 0 0"/>
-      <geometry>
-        <cylinder radius="0.065" length="0.04"/>
-      </geometry>
-    </visual>
-    <collision>
-      <origin xyz="0 0 0" rpy="1.5708 0 0"/>
-      <geometry>
-        <cylinder radius="0.065" length="0.04"/>
-      </geometry>
-    </collision>
-    <inertial>
-      <mass value="0.25"/>
-      <inertia ixx="0.0001" ixy="0" ixz="0" iyy="0.0001" iyz="0" izz="0.0001"/>
-    </inertial>
-  </link>
-  <link name="right_wheel_link">
-    <visual>
-      <origin xyz="0 0 0" rpy="1.5708 0 0"/>
-      <geometry>
-        <cylinder radius="0.065" length="0.04"/>
-      </geometry>
-    </visual>
-    <collision>
-      <origin xyz="0 0 0" rpy="1.5708 0 0"/>
-      <geometry>
-        <cylinder radius="0.065" length="0.04"/>
-      </geometry>
-    </collision>
-    <inertial>
-      <mass value="0.25"/>
-      <inertia ixx="0.0001" ixy="0" ixz="0" iyy="0.0001" iyz="0" izz="0.0001"/>
-    </inertial>
-  </link>
-  <joint name="left_wheel_joint" type="continuous">
-    <parent link="base_link"/>
-    <child link="left_wheel_link"/>
-    <origin xyz="0 0.17 0.065" rpy="0 0 0"/>
-    <axis xyz="0 1 0"/>
-  </joint>
-  <joint name="right_wheel_joint" type="continuous">
-    <parent link="base_link"/>
-    <child link="right_wheel_link"/>
-    <origin xyz="0 -0.17 0.065" rpy="0 0 0"/>
-    <axis xyz="0 1 0"/>
-  </joint>
-  <ros2_control name="TestDDBotHardware" type="system">
-    <hardware>
-      <plugin>test_dd_bot_hardware/TestDDBotHardware</plugin>
-      <param name="serial_port">/dev/ttyACM0</param>
-      <param name="baud_rate">9600</param>
-      <param name="wheel_radius">0.065</param>
-      <param name="wheel_base">0.34</param>
-    </hardware>
-    <joint name="left_wheel_joint">
-      <command_interface name="velocity"/>
-      <state_interface name="position"/>
-      <state_interface name="velocity"/>
+    <xacro:arg name="prefix" default="" />
+    <material name="blue">
+        <color rgba="0.0 0.4 0.8 1" />
+    </material>
+    <link name="base_link">
+        <visual>
+            <origin xyz="0 0 0.05" rpy="0 0 0" />
+            <geometry>
+                <box size="0.35 0.22 0.10" />
+            </geometry>
+            <material name="blue" />
+        </visual>
+        <collision>
+            <origin xyz="0 0 0.05" rpy="0 0 0" />
+            <geometry>
+                <box size="0.35 0.22 0.10" />
+            </geometry>
+        </collision>
+        <inertial>
+            <origin xyz="0 0 0.05" rpy="0 0 0" />
+            <mass value="2.0" />
+            <inertia ixx="0.01" ixy="0" ixz="0" iyy="0.02" iyz="0" izz="0.03" />
+        </inertial>
+    </link>
+    <link name="left_wheel_link">
+        <visual>
+            <origin xyz="0 0 0" rpy="1.5708 0 0" />
+            <geometry>
+                <cylinder radius="0.065" length="0.04" />
+            </geometry>
+        </visual>
+        <collision>
+            <origin xyz="0 0 0" rpy="1.5708 0 0" />
+            <geometry>
+                <cylinder radius="0.065" length="0.04" />
+            </geometry>
+        </collision>
+        <inertial>
+            <mass value="0.25" />
+            <inertia ixx="0.0001" ixy="0" ixz="0" iyy="0.0001" iyz="0" izz="0.0001" />
+        </inertial>
+    </link>
+    <link name="right_wheel_link">
+        <visual>
+            <origin xyz="0 0 0" rpy="1.5708 0 0" />
+            <geometry>
+                <cylinder radius="0.065" length="0.04" />
+            </geometry>
+        </visual>
+        <collision>
+            <origin xyz="0 0 0" rpy="1.5708 0 0" />
+            <geometry>
+                <cylinder radius="0.065" length="0.04" />
+            </geometry>
+        </collision>
+        <inertial>
+            <mass value="0.25" />
+            <inertia ixx="0.0001" ixy="0" ixz="0" iyy="0.0001" iyz="0" izz="0.0001" />
+        </inertial>
+    </link>
+    <joint name="left_wheel_joint" type="continuous">
+        <parent link="base_link" />
+        <child link="left_wheel_link" />
+        <origin xyz="0 0.17 0.065" rpy="0 0 0" />
+        <axis xyz="0 1 0" />
     </joint>
-    <joint name="right_wheel_joint">
-      <command_interface name="velocity"/>
-      <state_interface name="position"/>
-      <state_interface name="velocity"/>
+    <joint name="right_wheel_joint" type="continuous">
+        <parent link="base_link" />
+        <child link="right_wheel_link" />
+        <origin xyz="0 -0.17 0.065" rpy="0 0 0" />
+        <axis xyz="0 1 0" />
     </joint>
-  </ros2_control>
+    <ros2_control name="TestDDBotHardware" type="system">
+        <hardware>
+            <plugin>test_dd_bot_hardware/TestDDBotHardware</plugin>
+            <param name="serial_port">/dev/ttyACM0</param>
+            <param name="baud_rate">9600</param>
+            <param name="wheel_radius">0.065</param>
+            <param name="wheel_base">0.34</param>
+        </hardware>
+        <joint name="left_wheel_joint">
+            <command_interface name="velocity" />
+            <state_interface name="position" />
+            <state_interface name="velocity" />
+        </joint>
+        <joint name="right_wheel_joint">
+            <command_interface name="velocity" />
+            <state_interface name="position" />
+            <state_interface name="velocity" />
+        </joint>
+    </ros2_control>
 </robot>
